Commit message: 1.0.6

File: roch_description/urdf/sensors/rplidar.urdf.xacro (robot description, xacro)
@@ -25,10 +25,10 @@
 SOFTWARE, EVEN IF ADVISED OF THE POSSIBILITY OF SUCH DAMAGE.
 -->
-<robot xmlns:xacro="http://ros.org/wiki/xacro" name="ls_ls01c">
+<robot xmlns:xacro="http://ros.org/wiki/xacro" name="rplidar">
   <xacro:property name="laser_x" value="0.08" />
   <xacro:property name="laser_y" value="0.08" />
   <xacro:property name="laser_z" value="0.05526" />
   <xacro:property name="laser_mass" value=".1" />
-  <xacro:macro name="ls_ls01c" params="parent:=base_link">
+  <xacro:macro name="rplidar" params="parent:=base_link">
     <link name="base_laser_link">
       <inertial>
@@ -42,5 +42,5 @@
         <origin xyz="0 0 0" rpy="0 0 0" />
         <geometry>
-          <mesh filename="package://roch_description/meshes/sensors/ls_01c.stl" />
+          <mesh filename="package://roch_description/meshes/sensors/rplidar.stl" />
         </geometry>
         <xacro:insert_block name="roch_dark_grey" />
@@ -60,5 +60,5 @@
     <link name="base_laser"/>
     <joint name="base_laser_joint" type="fixed">
-      <origin xyz="0 0 0.04076" rpy=" ${M_PI} 0 0" />
+      <origin xyz="0 0 0.04076" rpy=" 0 ${M_PI} 0" />
       <parent link="base_laser_link" />
       <child link="base_laser" />
